Commit message: Clearned up the urdf files

File: simulation/robot_description/urdf/suction.urdf.xacro (robot description, xacro)
@@ -295,27 +295,6 @@
       <origin xyz="0.0 ${wrist_3_length} 0.0" rpy="-1.5707 0.0 0.0" />
     </joint>
-<!--
-    <joint name="${prefix}ee_fixed_joint" type="fixed">
-      <parent link="${prefix}wrist_3_link" />
-      <child link = "${prefix}ee_link" />
-      <origin xyz="0.0 ${wrist_3_length} 0.0" rpy="0.0 0.0 ${pi/2.0}" />
-    </joint>
-    <link name="${prefix}ee_link">
-      <collision>
-        <geometry>
-          <box size="0.01 0.01 0.01"/>
-        </geometry>
-        <surface>
-          <friction>
-            <ode>
-              <mu>10</mu>
-              <mu2>10</mu2>
-            </ode>
-          </friction>
-        </surface>
-        <origin rpy="0 0 0" xyz="-0.01 0 0"/>
-      </collision>
-    </link>  -->
-<!-- Vaccumm -->
+<!-- Vaccuum elements put at the tip of the nutdriver to simulate magnetic tip -->
+<!-- First Vacuum -->
     <link name="vacuum_gripper">
       <gravity>0</gravity>
@@ -343,4 +322,5 @@
       <dynamics damping="0.0" friction="10"/>
     </joint>
+<!-- Vaccuum plugin -->
   <gazebo>
       <plugin name="gazebo_ros_vacuum_gripper" filename="libgazebo_ros_vacuum_gripper.so">
@@ -353,5 +333,5 @@
       </plugin>
   </gazebo>
-<!-- second vacum -->
+<!-- Second vacuum -->
     <link name="vacuum_gripper1">
       <gravity>0</gravity>
@@ -389,5 +369,5 @@
       </plugin>
   </gazebo>
-<!-- third vacum -->
+<!-- Third vacuum -->
     <link name="vacuum_gripper2">
       <gravity>0</gravity>
@@ -425,5 +405,5 @@
       </plugin>
   </gazebo>
-<!-- include RAIL -->
+<!-- 7th axis linear rail -->
 <link name = "rail">
 <visual>
@@ -448,5 +428,5 @@
     </inertial>
   </link>
-<!-- Include Stands  -->
+<!-- Stand to elevate the rail for above manipulation  -->
 <link name = "rail_leg_1">
 <visual>

File: simulation/robot_description/urdf/suction_joint_limited_robot.urdf.xacro (robot description, xacro)
@@ -9,10 +9,4 @@
   <xacro:ur5_robot prefix="" joint_limited="true"/>
   <link name="world" />
-<!--
-  <joint name="world_joint" type="fixed">
-    <parent link="world" />
-    <child link = "base_link" />
-    <origin xyz="0.0 0.0 0.0" rpy="0.0 0.0 0.0" />
-  </joint> -->
   <joint name="world_joint" type="fixed">
     <parent link="world" />

File: simulation/robot_description/urdf/ur5.urdf.xacro (robot description, xacro)
@@ -285,26 +285,5 @@
       </collision>
     </link>
-<!-- include RAIL -->
-<!--
-<link name = "rail">
-<visual>
-      <geometry>
-        <box size="5 0.25 0.1"/>
-      </geometry>
-      <material name="LightGrey">
-        <color rgba="0.7 0.7 0.7 1.0"/>
-      </material>
- </visual>
-    <collision>
-      <geometry>
-        <box size="5 0.25 0.1"/>
-      </geometry>
-    </collision>
-    <inertial>
-      <mass value="15"/>
-      <origin rpy="0 0 0" xyz="0.0 0.0 0.0"/>
-      <inertia ixx="0.090625" ixy="0.0" ixz="0.0" iyy="31.26" iyz="0.0" izz="31.328"/>
-    </inertial>
-  </link>  -->
+<!-- 7th axis linear rail -->
 <link name = "rail">
 <visual>

File: simulation/robot_description/urdf/ur5_above_manipulation.urdf.xacro (robot description, xacro)
@@ -285,5 +285,5 @@
       </collision>
     </link>
-<!-- include RAIL -->
+<!-- 7th axis linear rail -->
 <link name = "rail">
 <visual>
@@ -308,5 +308,5 @@
     </inertial>
   </link>
-<!-- Include Stands  -->
+<!-- Stands to elevate the rail for above manipulation  -->
 <link name = "rail_leg_1">
 <visual>

File: simulation/robot_description/urdf/ur5_above_manipulation_gripper.urdf.xacro (robot description, xacro)
@@ -3,5 +3,5 @@
   <xacro:include filename="$(find robot_description)/urdf/ur5_above_manipulation_joint_limited_robot.urdf.xacro" />
   <xacro:include filename="$(find robotiq_description)/urdf/robotiq_85_gripper.urdf.xacro" />
- <!-- Robotiq Coupler -->
+  <!-- Robotiq Coupler -->
   <!--  + Height added by the coupler: 8mm -->
   <!--  + Reference frame: at the middle (4mm) -->
@@ -35,11 +35,4 @@
     <material>Gazebo/FlatBlack</material>
   </gazebo>
-  <!-- Equivalent to the OpenRAVE manipulator denso_robotiq_85_gripper -->
-  <!-- <link name="denso_robotiq_85_gripper" /> -->
-  <!-- <joint name="manipulator_dummy_joint" type="fixed"> -->
-  <!--   <origin xyz="0 0 0.1441" rpy="0 0 0" /> -->
-  <!--   <parent link="robotiq_coupler"/> -->
-  <!--   <child link="denso_robotiq_85_gripper"/> -->
-  <!-- </joint> -->
   <!-- Attach the robotiq 85 gripper -->
   <xacro:robotiq_85_gripper prefix="" parent="robotiq_coupler" >
@@ -59,4 +52,7 @@
   </gazebo>
   <!-- Gazebo grasping plugin -->
+<!-- Be sure to download plugin -->
+<!-- $ git clone https://github.com/JenniferBuehler/general-message-pkgs.git -->
+<!-- $ git clone https://github.com/JenniferBuehler/gazebo-pkgs.git -->
 <gazebo>
    <plugin name="gazebo_grasp_fix" filename="libgazebo_grasp_fix.so">

File: simulation/robot_description/urdf/ur5_above_manipulation_joint_limited_robot.urdf.xacro (robot description, xacro)
@@ -9,10 +9,4 @@
   <xacro:ur5_robot prefix="" joint_limited="true"/>
   <link name="world" />
-<!--
-  <joint name="world_joint" type="fixed">
-    <parent link="world" />
-    <child link = "base_link" />
-    <origin xyz="0.0 0.0 0.0" rpy="0.0 0.0 0.0" />
-  </joint> -->
   <joint name="world_joint" type="fixed">
     <parent link="world" />

File: simulation/robot_description/urdf/ur5_joint_limited_robot.urdf.xacro (robot description, xacro)
@@ -8,11 +8,4 @@
   <!-- arm -->
   <xacro:ur5_robot prefix="" joint_limited="true"/>
-<!-- with out laser
-  <link name="world" />
-  <joint name="world_joint" type="fixed">
-    <parent link="world" />
-    <child link = "rail" />
-    <origin xyz="0.0 0.0 0.0" rpy="0.0 0.0 0.0" />
-  </joint> -->
   <link name="base_footprint" />
   <joint name="world_joint" type="fixed">

File: simulation/robot_description/urdf/ur5_robot_above_manipulation.urdf.xacro (robot description, xacro)
@@ -2,4 +2,8 @@
 <robot name="ur5" xmlns:xacro="http://www.ros.org/wiki/xacro">
   <xacro:include filename="$(find robot_description)/urdf/ur5_above_manipulation_joint_limited_robot.urdf.xacro" />
+<!-- This urdf file is called from ur5_above_manipulation_setup.launch -->
+<!-- allows the user to enter the argument 'nut' -->
+<!-- if nut = true, then UR5 will be equipped with a nutdriver -->
+<!-- if nut == false (default) then UR5 will be equipped with a gripper -->
   <xacro:arg name="nut" default="false" />
   <xacro:property name="nut" value="$(arg nut)" />
@@ -28,5 +32,5 @@
       <origin xyz="0.0 0.0823 0.0" rpy="-1.5707 0.0 0.0" />
     </joint>
-<!-- Vaccumm -->
+<!-- Attach Vaccuum grippers to the tip of the nutdriver -->
     <link name="vacuum_gripper">
       <gravity>0</gravity>
@@ -64,5 +68,5 @@
       </plugin>
   </gazebo>
-<!-- second vacum -->
+<!-- second vacuum -->
     <link name="vacuum_gripper1">
       <gravity>0</gravity>
@@ -100,5 +104,5 @@
       </plugin>
   </gazebo>
-<!-- third vacum -->
+<!-- third vacuum -->
     <link name="vacuum_gripper2">
       <gravity>0</gravity>
@@ -136,5 +140,5 @@
       </plugin>
   </gazebo>
-    </xacro:if>
+ </xacro:if>
     <xacro:unless value="$(arg nut)">
   <xacro:include filename="$(find robotiq_description)/urdf/robotiq_85_gripper.urdf.xacro" />
@@ -171,11 +175,4 @@
     <material>Gazebo/FlatBlack</material>
   </gazebo>
-  <!-- Equivalent to the OpenRAVE manipulator denso_robotiq_85_gripper -->
-  <!-- <link name="denso_robotiq_85_gripper" /> -->
-  <!-- <joint name="manipulator_dummy_joint" type="fixed"> -->
-  <!--   <origin xyz="0 0 0.1441" rpy="0 0 0" /> -->
-  <!--   <parent link="robotiq_coupler"/> -->
-  <!--   <child link="denso_robotiq_85_gripper"/> -->
-  <!-- </joint> -->
   <!-- Attach the robotiq 85 gripper -->
   <xacro:robotiq_85_gripper prefix="" parent="robotiq_coupler" >
@@ -195,4 +192,6 @@
   </gazebo>
   <!-- Gazebo grasping plugin -->
+<!-- $ git clone https://github.com/JenniferBuehler/general-message-pkgs.git
+$ git clone https://github.com/JenniferBuehler/gazebo-pkgs.git -->
 <gazebo>
    <plugin name="gazebo_grasp_fix" filename="libgazebo_grasp_fix.so">

File: simulation/robot_description/urdf/ur5_robotiq85_gripper.urdf.xacro (robot description, xacro)
@@ -37,43 +37,9 @@
     <material>Gazebo/FlatBlack</material>
   </gazebo>
-<!--
-  <joint name="world_joint_2" type="fixed">
-    <parent link="base_footprint" />
-    <child link = "base_laser" />
-    <origin xyz="-2.4 -0.8 0.3" rpy="0.0 0.0 0.0" />
-  </joint>
-  <link name="base_laser" >
-    <visual>
-      <origin rpy="0 0 0" xyz="0.0 0.0 0.0"/>
-      <geometry>
-        <box size="0.05 0.05 0.6" />
-      </geometry>
-    </visual>
-    <collision>
-      <origin rpy="0 0 0" xyz="0.0 0.0 0.0"/>
-      <geometry>
-        <box size="0.05 0.05 0.6" />
-      </geometry>
-    </collision>
-    <inertial>
-      <origin xyz="0 0.0 0.15"/>
-      <mass value="10"/>
-      <inertia ixx="3.0" ixy="0.0" ixz="0.0"
-               iyy="3.0" iyz="0.0"
-               izz="3.0" />
-    </inertial>
-  </link>
--->
+<!-- Include 3D lidar laser -->
   <xacro:include filename="$(find robot_description)/urdf/VLP-16.urdf.xacro"/>
   <xacro:VLP-16 parent="base_footprint" name="velodyne" topic="/velodyne_points" hz="10" samples="440" gpu="${gpu}">
     <origin xyz="0.0 -0.3 0.5" rpy="0 0 0" />
   </xacro:VLP-16>
-  <!-- Equivalent to the OpenRAVE manipulator denso_robotiq_85_gripper -->
-  <!-- <link name="denso_robotiq_85_gripper" /> -->
-  <!-- <joint name="manipulator_dummy_joint" type="fixed"> -->
-  <!--   <origin xyz="0 0 0.1441" rpy="0 0 0" /> -->
-  <!--   <parent link="robotiq_coupler"/> -->
-  <!--   <child link="denso_robotiq_85_gripper"/> -->
-  <!-- </joint> -->
   <!-- Attach the robotiq 85 gripper -->
   <xacro:robotiq_85_gripper prefix="" parent="robotiq_coupler" >
